File: kicad/power_supply/power_supply.kicad_pcb (KiCad board)
At the start: 2 copper layers, 106.9 x 48 mm, 23 parts, among them J1 AC1, J2 GND, J3 CT, J4 AC2, J5 V-, J6 V+

Commit message: Power supply work
Parts:
- removed C3, C4: 100n, Capacitor_THT:C_Rect_L7.2mm_W5.5mm_P5.00mm_FKS2_FKP2_MKS2_MKP2
- removed the REF** at (165.6, 104.7)
- removed the REF** at (67.3, 66.3)
- removed the REF** at (67.3, 104.6)
- added C7: 4700u, Capacitor_THT:CP_Radial_D18.0mm_P7.50mm, F.Cu at (155.7, 72.1)
- added C8: 4700u, Capacitor_THT:CP_Radial_D18.0mm_P7.50mm, F.Cu at (155.7, 93.1)
- added J7: GND, TerminalBlock_Phoenix:TerminalBlock_Phoenix_MKDS-1,5-2_1x02_P5.00mm_Horizontal, F.Cu at (185.0, 88.4)
- added REF**: MountingHole_3.2mm_M3, MountingHole:MountingHole_3.2mm_M3, F.Cu at (186.2, 104.6)
- added REF**: MountingHole_3.2mm_M3, MountingHole:MountingHole_3.2mm_M3, F.Cu at (67.3, 66.3)
- added REF**: MountingHole_3.2mm_M3, MountingHole:MountingHole_3.2mm_M3, F.Cu at (67.3, 104.6)
- moved REF** 20.6 mm to (186.2, 65.8)
- moved J5 17.1 mm to (164.7, 101.6), turned to 90 degrees
- moved J3 14.2 mm to (164.7, 85.9), turned to 90 degrees
- moved J6 13.3 mm to (164.7, 70.9), turned to 90 degrees
- moved J5 13.3 mm to (171.2, 101.6), turned to 90 degrees
- moved J3 9.37 mm to (171.2, 85.9), turned to 90 degrees
- moved J1 7.88 mm to (69.6, 91.9)
- moved J6 7.88 mm to (171.2, 70.9), turned to 90 degrees
- moved J2 3.71 mm to (69.8, 80.3)
- moved C5 0.51 mm to (135.1, 72.3)
- moved C6 0.51 mm to (135.1, 93.0)
Routing:
- net /V+: track 94.2 -> 0.00 mm
- net /V-: track 93.7 -> 0.00 mm
- net /AC1: track 44.4 -> 41.2 mm
- added copper zone on B.Cu, net /V+
- added copper zone on B.Cu, net /V-
Other:
- board size 106.9 x 48 mm -> 129 x 48 mm
- board text removed: "Designed by Pontus Rydin. https://github.com/prydin/classab-amp-mosfet"
