File: kicad/power_supply/power_supply.kicad_sch (KiCad schematic)
At the start: 16 parts, among them J1 AC1, J2 GND, J3 CT, J4 AC2, J5 V-, J6 V+

Commit message: Power supply work
Parts:
- added C7, C8: 4700u, Capacitor_THT:CP_Radial_D18.0mm_P7.50mm, symbol Device:C_Polarized
- added J7: GND, TerminalBlock_Phoenix:TerminalBlock_Phoenix_MKDS-1,5-2_1x02_P5.00mm_Horizontal, symbol Connector:Screw_Terminal_01x02
Connections:
- net GND: now also C7.2, C8.1, J7.1 (Pin_1), J7.2 (Pin_2)
- net V+: now also C7.1
- net V-: now also C8.2
Other:
- moved on the sheet: C3, C4, J2, J5, J6
