File: kicad/classab-amp.kicad_sch (KiCad schematic)
At the start: 71 parts, among them J3 INPUT, Q1 2N5401, Q10 IRFP9240, Q11 2N5551, Q12 2N5551, Q13 BD139, Q14 BD140, Q15 2N5551, Q16 BD140, Q2 2N5401, Q3 2N5401, Q4 2N5401, Q5 2N5551, Q6 2N5401, Q7 BD139, Q8 BD139, Q9 IRFP240

Commit message: Release candidate 1
Parts:
- removed C14: 4700u, Capacitor_THT:CP_Radial_D18.0mm_P7.50mm, symbol Device:C_Polarized
- removed D1: 1N4148, Diode_THT:D_DO-35_SOD27_P5.08mm_Vertical_KathodeUp, symbol Diode:1N4148
- added C12: 220u, Capacitor_THT:CP_Radial_D8.0mm_P5.00mm, symbol Device:C_Polarized
- C13: value 4700u -> 220u; footprint Capacitor_THT:CP_Radial_D18.0mm_P7.50mm -> Capacitor_THT:CP_Radial_D8.0mm_P5.00mm
- R3, R5: value 470 -> 100
- R4: value 1k -> 470
Connections:
- net B+: now also C12.1
- net GNDS: now also J3.2 (Pin_2); no longer J3.1 (Pin_1)
- net PWRGND: now also C12.2
- net at C1.1: now also J3.1 (Pin_1); no longer J3.2 (Pin_2)
- net LTP COM: no longer names the net of Q2.1 (E), R25.2
Other:
- moved on the sheet: J3

Commit message: Update classab-amp.kicad_sch
Parts:
- C5: value 33p -> 47p
Changed lines of the file:
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@@
 			)
 		)
-		(property "Value" "33p"
+		(property "Value" "47p"
 			(at 133.35 110.744 90)
 			(effects

Commit message: V1.1
Parts:
- removed R22: 100, Resistor_THT:R_Axial_DIN0204_L3.6mm_D1.6mm_P7.62mm_Horizontal, symbol Device:R
- added J2: VOLUME, TerminalBlock_4Ucon:TerminalBlock_4Ucon_1x03_P3.50mm_Horizontal, symbol Connector:Screw_Terminal_01x03
- added R2: 100, Resistor_THT:R_Axial_DIN0204_L3.6mm_D1.6mm_P7.62mm_Horizontal, symbol Device:R
- added R3: 470, Resistor_THT:R_Axial_DIN0204_L3.6mm_D1.6mm_P7.62mm_Horizontal, symbol Device:R
- C1: renamed from C2; value 100p -> 220p
- C8: renamed from C9; value 68p -> 47p
- C9: renamed from C10; value 68p -> 47p
- R1: value 150 -> 1k
- R19: renamed from R10; value 47 -> 56
- R20: renamed from R6; value 22 -> 33
- renumbered C8 to C10, C16 to C11, C15 to C12, C12 to C13, C13 to C14, C3 to C15, C7 to C2, C1 to C3, C11 to C5, C5 to C6, C6 to C7, D8 to D1, D9 to D2, D2 to D3, D3 to D4, D4 to D5, D5 to D6, D6 to D7, D7 to D8, D10 to D9, J3 to J1, J2 to J3, J1 to J5, J5 to J6, J6 to J7, Q4 to Q1, Q16 to Q10, Q7 to Q11, Q8 to Q12, Q9 to Q15, Q10 to Q16, Q1 to Q2, Q11 to Q3, Q3 to Q4, Q2 to Q6, Q15 to Q7, Q12 to Q8, Q6 to Q9, R25 to R10, R5 to R11, R7 to R12, R9 to R14, R14 to R15, R11 to R17, R12 to R18, R23 to R21, R8 to R22, R18 to R23, R20 to R24, R2 to R4, R19 to R5, R15 to R6, R3 to R7, R24 to R8, R4 to R9
Connections:
- net GNDS: now also C1.2, C4.2, D3.2 (A), J1.1 (Pin_1), R4.1, J2.1 (Pin_1), R2.1; no longer J1.2 (Pin_2)
- net PWRGND: now also R2.2; no longer C1.2, C4.2, D3.2 (A), R4.1
- net at D1.2 (A), D2.1 (K), Q2.2 (B)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: now also C3.1; no longer C1.1, R1.2
- net at C3.2: now also R3.2; no longer R1.1
- new net: C1.1, J2.3 (Pin_3), R1.1
- new net: J2.2 (Pin_2), R3.1
- new net: J1.2 (Pin_2), R1.2
Other:
- moved on the sheet: C1, C3, J1, Q7, R1, R4

Commit message: Cleaned up SPICE, minor adjustments
Parts:
- R22, R23: value 47 -> 56
Changed lines of the file:
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@@
 			)
 		)
-		(property "Value" "47"
+		(property "Value" "56"
 			(at 190.5 40.64 90)
 			(effects
@@
 			)
 		)
-		(property "Value" "47"
+		(property "Value" "56"
 			(at 191.77 124.46 90)
 			(effects
